File: pcb/eink.kicad_pcb (KiCad board)
At the start: 2 copper layers, 42.2 x 65.3 mm, 30 parts, among them J1 USB_C_Receptacle_USB2.0_16P, J3 E-paper Display, SW1 SW_Push, SW2 RotaryEncoder_Switch, U1 ESP-12F, U3 RT6150AGQW, U4 CH340N

Commit message: pcb
Parts:
- removed REF** (x2): MountingHole_2.2mm_M2, MountingHole:MountingHole_2.2mm_M2
- added H1: MountingHole, MountingHole:MountingHole_2.2mm_M2, F.Cu at (175.2, 88.0)
- added H2: MountingHole, MountingHole:MountingHole_2.2mm_M2, F.Cu at (124.2, 88.0)
- added H3: MountingHole, MountingHole:MountingHole_2.2mm_M2, F.Cu at (124.2, 122.0)
- added H4: MountingHole, MountingHole:MountingHole_2.2mm_M2, F.Cu at (165.0, 122.2)
- C7: value C -> 10uF
- R5, R6: footprint Capacitor_SMD:C_0805_2012Metric -> Resistor_SMD:R_0805_2012Metric
- R8, R9: value R -> 5k1
- SW2: value RotaryEncoder_Switch -> RotaryEncoder_Switch_MP; footprint Rotary_Encoder:RotaryEncoder_Bourns_Vertical_PEC12R-3x17F-Sxxxx -> custom:EC11J
- moved R3 78.9 mm to (132.2, 114.8), turned to 90 degrees
- moved SW1 72.0 mm to (138.9, 111.1), turned to 0 degrees
- moved SW2 59.9 mm to (173.7, 115.6), turned to -90 degrees
- moved R2 59.7 mm to (151.4, 106.3), turned to 180 degrees
- moved L1 56.5 mm to (151.6, 117.9), turned to 180 degrees
- moved D7 54.9 mm to (160.4, 112.0)
- moved BT1 54.6 mm to (158.9, 123.0), turned to 180 degrees
- moved J3 54.1 mm to (127.2, 105.5)
- moved C1 52.8 mm to (134.9, 100.8)
- moved R4 52.4 mm to (135.0, 90.9), turned to 90 degrees
- moved C9 52.3 mm to (148.6, 114.4)
- moved U1 51.4 mm to (145.4, 89.3)
- moved C2 51.3 mm to (132.4, 100.8)
- moved R8 51.2 mm to (172.6, 105.8), turned to 180 degrees
- moved C8 51.0 mm to (154.6, 114.4), turned to 90 degrees
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Connections:
- C5 pad 1: Net-(U4-V3) -> VCC
- C6 pad 1: /RXD -> VCC
- D6 pad 2: /RXD -> Net-(D6-A)
- J1 pad A4: /RXD -> Net-(D6-A)
- J1 pad A9: /RXD -> Net-(D6-A)
- J1 pad B4: /RXD -> Net-(D6-A)
- J1 pad B9: /RXD -> Net-(D6-A)
- SW2 pad A: Net-(U1-GPIO4) -> Net-(U1-GPIO2)
- SW2 pad B: Net-(U1-GPIO2) -> Net-(U1-GPIO4)
- U1 pad 11: /CS -> /DC
- U1 pad 12: /DC -> /CS
- U1 pad 21: /RXD -> VCC
- U1 pad 22: /RXD -> VCC
- U4 pad 5: /RXD -> VCC
- U4 pad 6: /RXD -> VCC
- U4 pad 7: /RXD -> VCC
- U4 pad 8: Net-(U4-V3) -> VCC
Routing:
- net /RXD: track 72.3 -> 0.00 mm, vias 2 -> 0
- net /RESET: track 90.3 -> 69.3 mm, vias 0 -> 6
- net VCC: track 113.2 -> 93.3 mm, vias 2 -> 0
- net Net-(D6-A): track 0.00 -> 19.8 mm
- net Net-(U1-GPIO16): track 29.1 -> 48.8 mm
- net Net-(U1-GPIO0): track 6.27 -> 14.1 mm, vias 0 -> 2
- net Net-(U1-GPIO2): track 20.6 -> 28.4 mm
- net /DC: track 26.9 -> 19.5 mm
- net +BATT: track 16.0 -> 9.68 mm
- net GND: track 23.2 -> 27.9 mm, vias 10 -> 23
- net VBUS: track 5.08 -> 8.51 mm
- net Net-(U4-V3): track 2.96 -> 0.00 mm
- net Net-(U1-GPIO15): track 8.30 -> 5.62 mm
- net Net-(U3-FB): track 6.91 -> 4.59 mm
- net /BUSY: track 14.7 -> 13.0 mm
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- added copper zone on F.Cu, net VCC
Other:
- board size 42.2 x 65.3 mm -> 59 x 42 mm
